Commit message: URDF file working in rviz

File: src/base_package/models/base_robot.xacro (robot description, xacro)
@@ -1,27 +1,34 @@
 <?xml version="1.0"?>
-<robot xmlns:xacro="https://www.ros.org/wiki/xacro">
-<!-- <robot xmlns:drake="http://drake.mit.edu" name="ping_pong_arm"> -->
-    <!-- <xacro:property name="wrist_limit" value="${pi/2}"/> -->
+<robot xmlns:xacro="http://www.ros.org/wiki/xacro">
+    <xacro:include filename="inertial_macros.xacro"/>
+    <xacro:property name="upperarm_length" value="0.6" />
+    <xacro:property name="forearm_length" value="0.6" />
+    <xacro:property name="shoulder_height" value=".1" />
+    <xacro:property name="elbow_height" value="0.5" />
+    <material name="white">
+        <color rgba="1 1 1 1" />
+    </material>
     <link name="base_link"></link>
     <joint name="odrive_joint" type="fixed">
-        <parent link="base_link">
-        <child link="odrive_base">
+        <parent link="base_link"/>
+        <child link="odrive_base"/>
     </joint>
     <link name="odrive_base">
-        <inertial>
+        <!-- <inertial>
             <origin rpy="0 0 0" xyz="-0.1 0 0.07"/>
             <mass value="5"/>
             <inertia ixx="0.05" ixy="0" ixz="0" iyy="0.06" iyz="0" izz="0.03"/>
-        </inertial>
+        </inertial> -->
         <visual>
             <geometry>
-                <cylinder length="0.2" radius="0.06"/>
+                <cylinder length="${shoulder_height}" radius="0.06"/>
             </geometry>
-            <origin xyz="0 0 .1" />
             <material name="Black">
                 <color rgba="0 1.0 1.0 .50"/>
             </material>
+            <origin xyz="0 0 ${shoulder_height/2}"/>
         </visual>
-        <collision>
+        <xacro:inertial_pseudo/>
+        <!-- <collision>
             <origin rpy="0 0 0" xyz="-0.015 0 0.07"/>
             <geometry>
@@ -29,33 +36,29 @@
             </geometry>
             <material name="Grey"/>
-        </collision>
-        <!-- <self_collision_checking>
-            <origin rpy="0 0 0" xyz="0 0 0"/>
-            <geometry>
-                <capsule length="0.25" radius="0.15"/>
-            </geometry>
-        </self_collision_checking> -->
+        </collision> -->
     </link>
-    <joint name="shoulder" type="continuous">
+    <joint name="shoulder" type="revolute">
         <parent link="odrive_base"/>
-        <child link="upperarm"/>
-        <origin xyz="0 0 .2" rpy="1.57079632679 0 0"/>
-        <axis xyz="0 1 0" />
-        <limit drake:acceleration="8.57" effort="320" lower="-2.96705972839" upper="2.96705972839" velocity="1.4835298641951802"/>
-        <dynamics damping="0.5"/>
+        <child link="upper_arm"/>
+        <origin xyz="0 0 ${shoulder_height/2}"/>
+        <axis xyz="0 0 1" />
+        <limit upper="1.5" lower="-1.5" effort=".1" velocity=".5"/>
+        <!-- <limit drake:acceleration="8.57" effort="320" lower="-2.96705972839" upper="2.96705972839" velocity="1.4835298641951802"/>
+        <dynamics damping="0.5"/> -->
     </joint>
-    <link name="upperarm">
-        <inertial>
+    <link name="upper_arm">
+        <!-- <inertial>
             <origin rpy="0 0 0" xyz="0 -0.03 0.12"/>
             <mass value="5.76"/>
             <inertia ixx="0.033" ixy="0" ixz="0" iyy="0.0333" iyz="0" izz="0.0123"/>
-        </inertial>
+        </inertial> -->
         <visual>
             <geometry>
-                <box size=".04 .04 .3"/>
+                <box size=".04 ${upperarm_length} .04"/>
             </geometry>
-            <origin rpy="0 0 0" xyz="0 .02 .15" />
+            <origin xyz="0 ${upperarm_length/2} .02" />
         </visual>
-        <collision>
+        <xacro:inertial_pseudo/>
+        <!-- <collision>
             <origin rpy="0 0 0" xyz="0 -0.014 0.14"/>
             <geometry>
@@ -63,54 +66,5 @@
             </geometry>
             <material name="Grey"/>
-        </collision>
+        </collision> -->
     </link>
-    <!-- <link name="forearm">
-        <visual>
-            <geometry>
-                <box size=".04 .04 .3"/>
-            </geometry>
-            <origin xyz=".02 .04 .3"/>
-        </visual>
-    </link> -->
-    <!-- <joint name="base_joint" type="fixed">
-        <parent link="sidecar"/>
-        <child link="base"/>
-    </joint> -->
-    <!-- <joint name="elbow" type="continuous">
-        <origin xyz="0 0 0" rpy="0 0 0"/>
-        <parent link="upperarm"/>
-        <child link="forearm"/>
-    </joint> -->
-    <!-- <joint name="wrist_roll" type="revolute">
-        <origin xyz="5 0 0" rpy="0 0 0"/>
-        <axis xyz="1 0 0"/>
-        <parent link="forearm"/>
-        <child link="hand"/>
-        <limit lower="-1.57" upper="1.57"/>
-    </joint>
-    <joint name="wrist_pitch" type="revolute">
-        <origin xyz="5 0 0" rpy="0 0 0"/>
-        <axis xyz="0 1 0"/>
-        <parent link="forearm"/>
-        <child link="hand"/>
-        <limit lower="-1.57" upper="1.57"/>
-    </joint>
-    <joint name="wrist_yaw" type="revolute">
-        <origin xyz="5 0 0" rpy="0 0 0"/>
-        <axis xyz="0 0 1"/>
-        <parent link="forearm"/>
-        <child link="hand"/>
-        <limit lower="-1.57" upper="1.57"/>
-    </joint> -->
-    <!-- <transmission name="shoulder_transmission">
-        <robotNamespace>/iiwa</robotNamespace>
-        <type>transmission_interface/SimpleTransmission</type>
-        <joint name="shoulder">
-          <hardwareInterface>PositionJointInterface</hardwareInterface>
-        </joint>
-        <actuator name="shoulder_motor">
-          <hardwareInterface>PositionJointInterface</hardwareInterface>
-          <mechanicalReduction>1</mechanicalReduction>
-        </actuator>
-      </transmission> -->
-  </robot>
+</robot>

Commit message: simple URDF model complete

File: src/base_package/models/base_robot.xacro (robot description, xacro)
@@ -2,8 +2,10 @@
 <robot xmlns:xacro="http://www.ros.org/wiki/xacro">
     <xacro:include filename="inertial_macros.xacro"/>
+    <xacro:property name="shoulder_height" value="0.1" />
+    <xacro:property name="shoulder_radius" value="0.06" />
     <xacro:property name="upperarm_length" value="0.6" />
+    <xacro:property name="upperarm_width" value="0.04" />
     <xacro:property name="forearm_length" value="0.6" />
-    <xacro:property name="shoulder_height" value=".1" />
-    <xacro:property name="elbow_height" value="0.5" />
+    <xacro:property name="forearm_width" value="0.04" />
     <material name="white">
         <color rgba="1 1 1 1" />
@@ -22,5 +24,5 @@
         <visual>
             <geometry>
-                <cylinder length="${shoulder_height}" radius="0.06"/>
+                <cylinder length="${shoulder_height}" radius="${shoulder_radius}"/>
             </geometry>
             <material name="Black">
@@ -40,12 +42,12 @@
     <joint name="shoulder" type="revolute">
         <parent link="odrive_base"/>
-        <child link="upper_arm"/>
-        <origin xyz="0 0 ${shoulder_height/2}"/>
+        <child link="upperarm"/>
+        <origin xyz="0 0 ${shoulder_height}"/>
         <axis xyz="0 0 1" />
-        <limit upper="1.5" lower="-1.5" effort=".1" velocity=".5"/>
+        <limit upper="${pi/2}" lower="-${pi/2}" effort=".1" velocity=".5"/>
         <!-- <limit drake:acceleration="8.57" effort="320" lower="-2.96705972839" upper="2.96705972839" velocity="1.4835298641951802"/>
         <dynamics damping="0.5"/> -->
     </joint>
-    <link name="upper_arm">
+    <link name="upperarm">
         <!-- <inertial>
             <origin rpy="0 0 0" xyz="0 -0.03 0.12"/>
@@ -55,7 +57,37 @@
         <visual>
             <geometry>
-                <box size=".04 ${upperarm_length} .04"/>
+                <box size="${upperarm_width} ${upperarm_length} ${upperarm_width}"/>
             </geometry>
-            <origin xyz="0 ${upperarm_length/2} .02" />
+            <origin xyz="0 ${upperarm_length/2} ${upperarm_width/2}" />
+        </visual>
+        <xacro:inertial_pseudo/>
+        <!-- <collision>
+            <origin rpy="0 0 0" xyz="0 -0.014 0.14"/>
+            <geometry>
+              <cylinder length="0.29" radius="0.101"/>
+            </geometry>
+            <material name="Grey"/>
+        </collision> -->
+    </link>
+    <joint name="elbow" type="revolute">
+        <parent link="upperarm"/>
+        <child link="forearm"/>
+        <origin xyz="0 ${upperarm_length} ${upperarm_width}"/>
+        <axis xyz="0 0 1" />
+        <limit upper="${pi/2}" lower="-${pi/2}" effort=".1" velocity=".5"/>
+        <!-- <limit drake:acceleration="8.57" effort="320" lower="-2.96705972839" upper="2.96705972839" velocity="1.4835298641951802"/>
+        <dynamics damping="0.5"/> -->
+    </joint>
+    <link name="forearm">
+        <!-- <inertial>
+            <origin rpy="0 0 0" xyz="0 -0.03 0.12"/>
+            <mass value="5.76"/>
+            <inertia ixx="0.033" ixy="0" ixz="0" iyy="0.0333" iyz="0" izz="0.0123"/>
+        </inertial> -->
+        <visual>
+            <geometry>
+                <box size=".04 ${forearm_length} ${forearm_width}"/>
+            </geometry>
+            <origin xyz="0 ${forearm_length/2} ${forearm_width/2}" />
         </visual>
         <xacro:inertial_pseudo/>

Commit message: xacro improvements

File: src/base_package/models/base_robot.xacro (robot description, xacro)
@@ -2,13 +2,13 @@
 <robot xmlns:xacro="http://www.ros.org/wiki/xacro">
     <xacro:include filename="inertial_macros.xacro"/>
-    <xacro:property name="shoulder_height" value="0.1" />
-    <xacro:property name="shoulder_radius" value="0.06" />
-    <xacro:property name="upperarm_length" value="0.6" />
-    <xacro:property name="upperarm_width" value="0.04" />
-    <xacro:property name="forearm_length" value="0.6" />
-    <xacro:property name="forearm_width" value="0.04" />
-    <material name="white">
-        <color rgba="1 1 1 1" />
-    </material>
+    <xacro:include filename="visual_macros.xacro"/>
+    <xacro:property name="shoulder_radius" value="${.18/2}" />
+    <xacro:property name="shoulder_height" value=".1615" />
+    <xacro:property name="upperarm_length" value=".30381" />
+    <xacro:property name="upperarm_height" value="0.070471" />
+    <xacro:property name="upperarm_mass" value="0.4" />
+    <xacro:property name="forearm_length" value=".259916" />
+    <xacro:property name="forearm_height" value=".02545" />
+    <xacro:property name="forearm_mass" value="0.3" />
     <link name="base_link"></link>
     <joint name="odrive_joint" type="fixed">
@@ -17,26 +17,9 @@
     </joint>
     <link name="odrive_base">
-        <!-- <inertial>
-            <origin rpy="0 0 0" xyz="-0.1 0 0.07"/>
-            <mass value="5"/>
-            <inertia ixx="0.05" ixy="0" ixz="0" iyy="0.06" iyz="0" izz="0.03"/>
-        </inertial> -->
-        <visual>
-            <geometry>
-                <cylinder length="${shoulder_height}" radius="${shoulder_radius}"/>
-            </geometry>
-            <material name="Black">
-                <color rgba="0 1.0 1.0 .50"/>
+        <xacro:cylinder_identical_collision mass="3" radius="${shoulder_radius}" height="${shoulder_height}">
+            <material name="blue">
+                <color rgba="0 0 1 1" />
             </material>
-            <origin xyz="0 0 ${shoulder_height/2}"/>
-        </visual>
-        <xacro:inertial_pseudo/>
-        <!-- <collision>
-            <origin rpy="0 0 0" xyz="-0.015 0 0.07"/>
-            <geometry>
-              <cylinder length="0.17" radius="0.139"/>
-            </geometry>
-            <material name="Grey"/>
-        </collision> -->
+        </xacro:cylinder_identical_collision>
     </link>
     <joint name="shoulder" type="revolute">
@@ -50,28 +33,15 @@
     </joint>
     <link name="upperarm">
-        <!-- <inertial>
-            <origin rpy="0 0 0" xyz="0 -0.03 0.12"/>
-            <mass value="5.76"/>
-            <inertia ixx="0.033" ixy="0" ixz="0" iyy="0.0333" iyz="0" izz="0.0123"/>
-        </inertial> -->
-        <visual>
-            <geometry>
-                <box size="${upperarm_width} ${upperarm_length} ${upperarm_width}"/>
-            </geometry>
-            <origin xyz="0 ${upperarm_length/2} ${upperarm_width/2}" />
-        </visual>
-        <xacro:inertial_pseudo/>
-        <!-- <collision>
-            <origin rpy="0 0 0" xyz="0 -0.014 0.14"/>
-            <geometry>
-              <cylinder length="0.29" radius="0.101"/>
-            </geometry>
-            <material name="Grey"/>
-        </collision> -->
+        <xacro:square_prism_identical_collision mass="${upperarm_mass}" length="${upperarm_length}" height="${upperarm_height}">
+            <material name="green">
+                <color rgba="0 1 0 1" />
+            </material>
+        </xacro:square_prism_identical_collision>
+        <xacro:square_prism_inertial mass="${upperarm_mass}" length="${upperarm_length}" height="${upperarm_height}"/>
     </link>
     <joint name="elbow" type="revolute">
         <parent link="upperarm"/>
         <child link="forearm"/>
-        <origin xyz="0 ${upperarm_length} ${upperarm_width}"/>
+        <origin xyz="0 ${upperarm_length} ${upperarm_height}"/>
         <axis xyz="0 0 1" />
         <limit upper="${pi/2}" lower="-${pi/2}" effort=".1" velocity=".5"/>
@@ -80,23 +50,10 @@
     </joint>
     <link name="forearm">
-        <!-- <inertial>
-            <origin rpy="0 0 0" xyz="0 -0.03 0.12"/>
-            <mass value="5.76"/>
-            <inertia ixx="0.033" ixy="0" ixz="0" iyy="0.0333" iyz="0" izz="0.0123"/>
-        </inertial> -->
-        <visual>
-            <geometry>
-                <box size=".04 ${forearm_length} ${forearm_width}"/>
-            </geometry>
-            <origin xyz="0 ${forearm_length/2} ${forearm_width/2}" />
-        </visual>
-        <xacro:inertial_pseudo/>
-        <!-- <collision>
-            <origin rpy="0 0 0" xyz="0 -0.014 0.14"/>
-            <geometry>
-              <cylinder length="0.29" radius="0.101"/>
-            </geometry>
-            <material name="Grey"/>
-        </collision> -->
+        <xacro:square_prism_identical_collision mass="${forearm_mass}" length="${forearm_length}" height="${forearm_height}">
+            <material name="red">
+                <color rgba="1 1 0 1" />
+            </material>
+        </xacro:square_prism_identical_collision>
+        <xacro:square_prism_inertial mass="${forearm_mass}" length="${forearm_length}" height="${forearm_height}"/>
     </link>
 </robot>

File: src/base_package/models/inertial_macros.xacro (robot description, xacro)
@@ -1,10 +1,13 @@
 <?xml version="1.0"?>
 <robot xmlns:xacro="http://www.ros.org/wiki/xacro" >
-    <xacro:macro name="inertial_pseudo">
+    <!-- https://en.wikipedia.org/wiki/List_of_moments_of_inertia -->
+    <xacro:macro name="square_prism_inertial" params="mass length height">
         <inertial>
-            <mass value="1"/>
-            <inertia ixx="2" ixy="0.0" ixz="0.0"
-                    iyy="2" iyz="0.0"
-                    izz="2" />
+            <mass value="${mass}"/>
+            <!-- In the Articulated Robot video, his xyz here is x, 0, z. Why? -->
+            <origin xyz="${height/2} ${length/2} ${height/2}" />
+            <inertia ixx="${1/12 * mass * (length*length + height*height)}" ixy="0.0" ixz="0.0"
+                    iyy="${1/12 * mass * (2 * height*height)}" iyz="0.0"
+                    izz="${1/12 * mass * (length*length + height*height)}" />
         </inertial>
     </xacro:macro>
