Commit message: basic launch file working

File: src/base_package/models/helper/robot.ros2_control.xacro (robot description, xacro)
@@ -1,7 +1,8 @@
 <?xml version="1.0"?>
 <robot xmlns:xacro="http://www.ros.org/wiki/xacro">
-    <xacro:macro name="ros2_control_robot" params="name prefix">
+    <!-- <xacro:macro name="ros2_control_robot" params="name prefix"> -->
         <ros2_control name="louis_bot" type="system">
-            <hardware>
+            <!-- TODO: add custom controller here!! -->
+            <!-- <hardware>
                 <xacro:if value="${use_mode_mock_hardware}">
                     <plugin>mock_components/GenericSystem</plugin>
@@ -14,7 +15,9 @@
                 </xacro:if>
                 <xacro:unless value="${use_mode_mock_hardware or use_mode_classic_gazebo or use_mode_gazebo}">
-                    <!-- TODO: add custom controller here!! -->
                     <plugin>package_name/ClassName</plugin>
                 </xacro:unless>
+            </hardware> -->
+            <hardware>
+                <plugin>mock_components/GenericSystem</plugin>
             </hardware>
             <joint name="shoulder">
@@ -44,4 +47,4 @@
             </joint>
         </ros2_control>
-    </xacro:macro>
+    <!-- </xacro:macro> -->
 </robot>

Commit message: working forward controller rviz robot

File: src/base_package/models/helper/robot.ros2_control.xacro (robot description, xacro)
@@ -1,50 +1,53 @@
 <?xml version="1.0"?>
 <robot xmlns:xacro="http://www.ros.org/wiki/xacro">
-    <!-- <xacro:macro name="ros2_control_robot" params="name prefix"> -->
-        <ros2_control name="louis_bot" type="system">
-            <!-- TODO: add custom controller here!! -->
-            <!-- <hardware>
-                <xacro:if value="${use_mode_mock_hardware}">
-                    <plugin>mock_components/GenericSystem</plugin>
-                </xacro:if>
-                <xacro:if value="${use_mode_classic_gazebo}">
-                    <plugin>gazebo_ros2_control/GazeboSystem</plugin>
-                </xacro:if>
-                <xacro:if value="${use_mode_gazebo}">
-                    <plugin>ign_ros2_control/IgnitionSystem</plugin>
-                </xacro:if>
-                <xacro:unless value="${use_mode_mock_hardware or use_mode_classic_gazebo or use_mode_gazebo}">
-                    <plugin>package_name/ClassName</plugin>
-                </xacro:unless>
-            </hardware> -->
-            <hardware>
+    <ros2_control name="louis_bot" type="system">
+        <!-- TODO: add custom controller here!! -->
+        <!-- <hardware>
+            <xacro:if value="${use_mode_mock_hardware}">
                 <plugin>mock_components/GenericSystem</plugin>
-            </hardware>
-            <joint name="shoulder">
-                <!-- can use position or velocity port to connect a controller -->
-                <command_interface name="position">
-                    <param name="min">-1</param>
-                    <param name="max">1</param>
-                </command_interface>
-                <command_interface name="velocity">
-                    <param name="min">-1</param>
-                    <param name="max">1</param>
-                </command_interface>
-                <state_interface name="position"/>
-                <state_interface name="velocity"/>
-            </joint>
-            <joint name="elbow">
-                <command_interface name="position">
-                    <param name="min">-1</param>
-                    <param name="max">1</param>
-                </command_interface>
-                <command_interface name="velocity">
-                    <param name="min">-1</param>
-                    <param name="max">1</param>
-                </command_interface>
-                <state_interface name="position"/>
-                <state_interface name="velocity"/>
-            </joint>
-        </ros2_control>
-    <!-- </xacro:macro> -->
+            </xacro:if>
+            <xacro:if value="${use_mode_classic_gazebo}">
+                <plugin>gazebo_ros2_control/GazeboSystem</plugin>
+            </xacro:if>
+            <xacro:if value="${use_mode_gazebo}">
+                <plugin>ign_ros2_control/IgnitionSystem</plugin>
+            </xacro:if>
+            <xacro:unless value="${use_mode_mock_hardware or use_mode_classic_gazebo or use_mode_gazebo}">
+                <plugin>package_name/ClassName</plugin>
+            </xacro:unless>
+        </hardware> -->
+        <hardware>
+            <plugin>mock_components/GenericSystem</plugin>
+        </hardware>
+        <joint name="shoulder">
+            <!-- can use position or velocity port to connect a controller -->
+            <command_interface name="position">
+                <param name="min">-1</param>
+                <param name="max">1</param>
+            </command_interface>
+            <command_interface name="velocity">
+                <param name="min">-1</param>
+                <param name="max">1</param>
+            </command_interface>
+            <state_interface name="position"/>
+            <state_interface name="velocity"/>
+        </joint>
+        <joint name="elbow">
+            <command_interface name="position">
+                <param name="min">-1</param>
+                <param name="max">1</param>
+            </command_interface>
+            <command_interface name="velocity">
+                <param name="min">-1</param>
+                <param name="max">1</param>
+            </command_interface>
+            <state_interface name="position"/>
+            <state_interface name="velocity"/>
+        </joint>
+    </ros2_control>
+    <!-- <gazebo>
+        <plugin name="gazebo_ros2_control" filename="libgazebo_ros_diff_drive.so ">
+            <parameters>$(find base_package)/bringup/config/controller.yaml</parameters>
+        </plugin>
+    </gazebo> -->
 </robot>
