Commit message: controller changes

File: src/base_package/models/helper/base_robot.xacro (robot description, xacro)
@@ -11,4 +11,8 @@
     <xacro:property name="forearm_height" value=".02545" />
     <xacro:property name="forearm_mass" value="0.3" />
+    <xacro:property name="end_effector_radius" value="${.1/2}" />
+    <xacro:property name="end_effector_length" value="0.1" />
+    <xacro:property name="end_effector_height" value="0.02" />
+    <xacro:property name="end_effector_mass" value=".1" />
     <link name="base_link"></link>
     <joint name="odrive_joint" type="fixed">
@@ -52,8 +56,25 @@
         <xacro:square_prism_identical_collision mass="${forearm_mass}" length="${forearm_length}" height="${forearm_height}">
             <material name="red">
-                <color rgba="1 1 0 1" />
+                <color rgba="1 0 0 1" />
             </material>
         </xacro:square_prism_identical_collision>
         <xacro:square_prism_inertial mass="${forearm_mass}" length="${forearm_length}" height="${forearm_height}"/>
     </link>
+    <joint name="wrist" type="fixed">
+        <parent link="forearm"/>
+        <child link="end_effector"/>
+        <origin xyz="0 ${forearm_length} ${forearm_height}" rpy="-${pi/2} 0 0"/>
+        <axis xyz="0 0 1" />
+        <limit upper="${pi/2}" lower="-${pi/2}" effort=".1" velocity=".5"/>
+        <!-- <limit drake:acceleration="8.57" effort="320" lower="-2.96705972839" upper="2.96705972839" velocity="1.4835298641951802"/>
+        <dynamics damping="0.5"/> -->
+    </joint>
+    <link name="end_effector">
+        <xacro:square_prism_identical_collision mass="${end_effector_mass}" length="${end_effector_length}" height="${end_effector_height}">
+            <material name="orange">
+                <color rgba="1 0 1 1" />
+            </material>
+        </xacro:square_prism_identical_collision>
+        <xacro:square_prism_inertial mass="${end_effector_mass}" length="${end_effector_length}" height="${end_effector_height}"/>
+    </link>
 </robot>

Commit message: MESSY transmission

File: src/base_package/models/helper/base_robot.xacro (robot description, xacro)
@@ -47,5 +47,6 @@
         <parent link="upperarm"/>
         <child link="forearm"/>
-        <origin xyz="0 ${upperarm_length} ${upperarm_height}"/>
+        <!-- start at pi/2 so not at a singularity -->
+        <origin xyz="0 ${upperarm_length} ${upperarm_height}" rpy="0 0 ${pi/2}"/>
         <axis xyz="0 0 1" />
         <limit upper="${pi/2}" lower="-${pi/2}" effort=".1" velocity=".5"/>
@@ -78,3 +79,9 @@
         <xacro:square_prism_inertial mass="${end_effector_mass}" length="${end_effector_length}" height="${end_effector_height}"/>
     </link>
+    <!-- Drake 'MultibodyPlant does not currently support non-default mechanical reductions.' -->
+    <!-- <transmission name="transm" type="SimpleTransmission">
+        <joint name="shoulder"/>
+        <actuator name="shoulder_motor"/>
+        <mechanicalReduction>.1</mechanicalReduction>
+    </transmission> -->
 </robot>

File: src/base_package/models/helper/ros2_control_hardware_interfaces/mock.ros2_control.xacro (robot description, xacro)
@@ -30,4 +30,21 @@
             <!-- <state_interface name="velocity"/> -->
         </joint>
+        <!-- <transmission name="transmission1">
+            <plugin>transmission_interface/SimpleTransmission</plugin>
+            <actuator name="shoulder_actuator" role="shoulder_actuator"/>
+            <joint name="shoulder" role="shoulder">
+                31/30*w_s = 122/30*w_c
+                <mechanical_reduction>${122/31}</mechanical_reduction>
+                <offset>0.0</offset>
+            </joint>
+        </transmission>
+        <transmission name="transmission1">
+            <plugin>transmission_interface/SimpleTransmission</plugin>
+            <actuator name="elbow_actuator" role="elbow_actuator"/>
+            <joint name="elbow" role="elbow">
+                <mechanical_reduction>4.0</mechanical_reduction>
+                <offset>0.0</offset>
+            </joint>
+        </transmission> -->
     </ros2_control>
 </robot>

File: src/base_package/models/helper/ros2_control_hardware_interfaces/real.ros2_control.xacro (robot description, xacro)
@@ -11,4 +11,13 @@
             <param name="node_id">0</param>
         </joint>
+        <!-- <transmission name="transmission1"> -->
+            <!-- <plugin>transmission_interface/SimpleTransmission</plugin> -->
+            <!-- <actuator name="shoulder_actuator" role="shoulder_actuator"/> -->
+            <!-- <joint name="shoulder" role="shoulder"> -->
+                <!-- 31/30*w_s = 122/30*w_c ${31/122}-->
+                <!-- <mechanical_reduction>325</mechanical_reduction>
+                <offset>0.0</offset>
+            </joint>
+        </transmission> -->
     </ros2_control>
     <ros2_control name="elbow_interface" type="system">
@@ -26,4 +35,13 @@
             <state_interface name="position"/>
         </joint>
+        <!-- <transmission name="transmission1"> -->
+            <!-- <plugin>transmission_interface/SimpleTransmission</plugin> -->
+            <!-- <actuator name="elbow_actuator" role="elbow_actuator"/> -->
+            <!-- <joint name="elbow" role="elbow">
+                <mechanical_reduction>4.0</mechanical_reduction>
+                <offset>0.0</offset>
+            </joint>
+        </transmission>
+         -->
     </ros2_control>
 </robot>
